File: k34-plate/k34.kicad_pcb (KiCad board)
At the start: 2 copper layers, 254.2 x 118.9 mm, 6 parts

Commit message: added 3rd screw
Parts:
- removed the REF** at (155.2, 58.3)
- removed the REF** at (234.9, 52.1)
- removed the REF** at (184.5, 117.9)
- removed the REF** at (94.6, 117.9)
- removed the REF** at (123.7, 58.3)
- added REF**: MountingHole_2.2mm_M2, MountingHole:MountingHole_2.2mm_M2, F.Cu at (94.7, 106.8)
- added REF**: MountingHole_2.2mm_M2, MountingHole:MountingHole_2.2mm_M2, F.Cu at (105.9, 40.9)
- moved REF** 11.0 mm to (43.9, 40.9)
Other:
- board size 254.2 x 118.9 mm -> 113.5 x 118.9 mm
