File: k34/k34.sch (KiCad schematic (older format))
At the start: 69 parts, among them U1 nice_nano

Commit message: updated schematic with wider diode
Parts:
- D1, D10, D11, D12, D13, D14, D15, D16, D17, D18, D19, D2, D20, D21, D22, D23, D24, D25, D26, D27, D28, D29, D3, D30, D31, D32, D33, D34, D4, D5, D6, D7, D8, D9: footprint Diode_SMD:D_SOD-323_HandSoldering -> Diode_SMD:D_SOD-128
Changed lines of the file:
@@
 F 0 "D1" V 1846 2580 50  0000 R CNN
 F 1 "D_Small" V 1755 2580 50  0000 R CNN
-F 2 "Diode_SMD:D_SOD-323_HandSoldering" V 1800 2650 50  0001 C CNN
+F 2 "Diode_SMD:D_SOD-128" V 1800 2650 50  0001 C CNN
 F 3 "~" V 1800 2650 50  0001 C CNN
 	1    1800 2650
@@
 F 0 "D2" V 2346 2580 50  0000 R CNN
 F 1 "D_Small" V 2255 2580 50  0000 R CNN
-F 2 "Diode_SMD:D_SOD-323_HandSoldering" V 2300 2650 50  0001 C CNN
+F 2 "Diode_SMD:D_SOD-128" V 2300 2650 50  0001 C CNN
 F 3 "~" V 2300 2650 50  0001 C CNN
 	1    2300 2650
@@
 F 0 "D3" V 2846 2580 50  0000 R CNN
 F 1 "D_Small" V 2755 2580 50  0000 R CNN
-F 2 "Diode_SMD:D_SOD-323_HandSoldering" V 2800 2650 50  0001 C CNN
+F 2 "Diode_SMD:D_SOD-128" V 2800 2650 50  0001 C CNN
 F 3 "~" V 2800 2650 50  0001 C CNN
 	1    2800 2650
@@
 F 0 "D4" V 3346 2580 50  0000 R CNN
 F 1 "D_Small" V 3255 2580 50  0000 R CNN
-F 2 "Diode_SMD:D_SOD-323_HandSoldering" V 3300 2650 50  0001 C CNN
+F 2 "Diode_SMD:D_SOD-128" V 3300 2650 50  0001 C CNN
 F 3 "~" V 3300 2650 50  0001 C CNN
 	1    3300 2650
@@
 F 0 "D5" V 3846 2580 50  0000 R CNN
 F 1 "D_Small" V 3755 2580 50  0000 R CNN
-F 2 "Diode_SMD:D_SOD-323_HandSoldering" V 3800 2650 50  0001 C CNN
+F 2 "Diode_SMD:D_SOD-128" V 3800 2650 50  0001 C CNN
 F 3 "~" V 3800 2650 50  0001 C CNN
 	1    3800 2650
@@
 F 0 "D6" V 4346 2580 50  0000 R CNN
 F 1 "D_Small" V 4255 2580 50  0000 R CNN
-F 2 "Diode_SMD:D_SOD-323_HandSoldering" V 4300 2650 50  0001 C CNN
+F 2 "Diode_SMD:D_SOD-128" V 4300 2650 50  0001 C CNN
 F 3 "~" V 4300 2650 50  0001 C CNN
 	1    4300 2650
@@
 F 0 "D7" V 4846 2580 50  0000 R CNN
 F 1 "D_Small" V 4755 2580 50  0000 R CNN
-F 2 "Diode_SMD:D_SOD-323_HandSoldering" V 4800 2650 50  0001 C CNN
+F 2 "Diode_SMD:D_SOD-128" V 4800 2650 50  0001 C CNN
 F 3 "~" V 4800 2650 50  0001 C CNN
 	1    4800 2650
@@
 F 0 "D8" V 5346 2580 50  0000 R CNN
 F 1 "D_Small" V 5255 2580 50  0000 R CNN
-F 2 "Diode_SMD:D_SOD-323_HandSoldering" V 5300 2650 50  0001 C CNN
+F 2 "Diode_SMD:D_SOD-128" V 5300 2650 50  0001 C CNN
 F 3 "~" V 5300 2650 50  0001 C CNN
 	1    5300 2650
@@
 F 0 "D9" V 5846 2580 50  0000 R CNN
 F 1 "D_Small" V 5755 2580 50  0000 R CNN
-F 2 "Diode_SMD:D_SOD-323_HandSoldering" V 5800 2650 50  0001 C CNN
+F 2 "Diode_SMD:D_SOD-128" V 5800 2650 50  0001 C CNN
 F 3 "~" V 5800 2650 50  0001 C CNN
 	1    5800 2650
@@
 F 0 "D10" V 6346 2580 50  0000 R CNN
 F 1 "D_Small" V 6255 2580 50  0000 R CNN
-F 2 "Diode_SMD:D_SOD-323_HandSoldering" V 6300 2650 50  0001 C CNN
+F 2 "Diode_SMD:D_SOD-128" V 6300 2650 50  0001 C CNN
 F 3 "~" V 6300 2650 50  0001 C CNN
 	1    6300 2650
@@
 F 0 "D11" V 1846 3230 50  0000 R CNN
 F 1 "D_Small" V 1755 3230 50  0000 R CNN
-F 2 "Diode_SMD:D_SOD-323_HandSoldering" V 1800 3300 50  0001 C CNN
+F 2 "Diode_SMD:D_SOD-128" V 1800 3300 50  0001 C CNN
 F 3 "~" V 1800 3300 50  0001 C CNN
 	1    1800 3300
@@
 F 0 "D12" V 2346 3230 50  0000 R CNN
 F 1 "D_Small" V 2255 3230 50  0000 R CNN
-F 2 "Diode_SMD:D_SOD-323_HandSoldering" V 2300 3300 50  0001 C CNN
+F 2 "Diode_SMD:D_SOD-128" V 2300 3300 50  0001 C CNN
 F 3 "~" V 2300 3300 50  0001 C CNN
 	1    2300 3300
@@
 F 0 "D13" V 2846 3230 50  0000 R CNN
 F 1 "D_Small" V 2755 3230 50  0000 R CNN
-F 2 "Diode_SMD:D_SOD-323_HandSoldering" V 2800 3300 50  0001 C CNN
+F 2 "Diode_SMD:D_SOD-128" V 2800 3300 50  0001 C CNN
 F 3 "~" V 2800 3300 50  0001 C CNN
 	1    2800 3300
@@
 F 0 "D14" V 3346 3230 50  0000 R CNN
 F 1 "D_Small" V 3255 3230 50  0000 R CNN
-F 2 "Diode_SMD:D_SOD-323_HandSoldering" V 3300 3300 50  0001 C CNN
+F 2 "Diode_SMD:D_SOD-128" V 3300 3300 50  0001 C CNN
 F 3 "~" V 3300 3300 50  0001 C CNN
 	1    3300 3300
@@
 F 0 "D15" V 3846 3230 50  0000 R CNN
 F 1 "D_Small" V 3755 3230 50  0000 R CNN
-F 2 "Diode_SMD:D_SOD-323_HandSoldering" V 3800 3300 50  0001 C CNN
+F 2 "Diode_SMD:D_SOD-128" V 3800 3300 50  0001 C CNN
 F 3 "~" V 3800 3300 50  0001 C CNN
 	1    3800 3300
@@
 F 0 "D16" V 4346 3230 50  0000 R CNN
 F 1 "D_Small" V 4255 3230 50  0000 R CNN
-F 2 "Diode_SMD:D_SOD-323_HandSoldering" V 4300 3300 50  0001 C CNN
+F 2 "Diode_SMD:D_SOD-128" V 4300 3300 50  0001 C CNN
 F 3 "~" V 4300 3300 50  0001 C CNN
 	1    4300 3300
@@
 F 0 "D17" V 4846 3230 50  0000 R CNN
 F 1 "D_Small" V 4755 3230 50  0000 R CNN
-F 2 "Diode_SMD:D_SOD-323_HandSoldering" V 4800 3300 50  0001 C CNN
+F 2 "Diode_SMD:D_SOD-128" V 4800 3300 50  0001 C CNN
 F 3 "~" V 4800 3300 50  0001 C CNN
 	1    4800 3300
@@
 F 0 "D18" V 5346 3230 50  0000 R CNN
 F 1 "D_Small" V 5255 3230 50  0000 R CNN
-F 2 "Diode_SMD:D_SOD-323_HandSoldering" V 5300 3300 50  0001 C CNN
+F 2 "Diode_SMD:D_SOD-128" V 5300 3300 50  0001 C CNN
 F 3 "~" V 5300 3300 50  0001 C CNN
 	1    5300 3300
@@
 F 0 "D19" V 5846 3230 50  0000 R CNN
 F 1 "D_Small" V 5755 3230 50  0000 R CNN
-F 2 "Diode_SMD:D_SOD-323_HandSoldering" V 5800 3300 50  0001 C CNN
+F 2 "Diode_SMD:D_SOD-128" V 5800 3300 50  0001 C CNN
 F 3 "~" V 5800 3300 50  0001 C CNN
 	1    5800 3300
@@
 F 0 "D20" V 6346 3230 50  0000 R CNN
 F 1 "D_Small" V 6255 3230 50  0000 R CNN
-F 2 "Diode_SMD:D_SOD-323_HandSoldering" V 6300 3300 50  0001 C CNN
+F 2 "Diode_SMD:D_SOD-128" V 6300 3300 50  0001 C CNN
 F 3 "~" V 6300 3300 50  0001 C CNN
 	1    6300 3300
@@
 F 0 "D21" V 1846 3880 50  0000 R CNN
 F 1 "D_Small" V 1755 3880 50  0000 R CNN
-F 2 "Diode_SMD:D_SOD-323_HandSoldering" V 1800 3950 50  0001 C CNN
+F 2 "Diode_SMD:D_SOD-128" V 1800 3950 50  0001 C CNN
 F 3 "~" V 1800 3950 50  0001 C CNN
 	1    1800 3950
@@
 F 0 "D22" V 2346 3880 50  0000 R CNN
 F 1 "D_Small" V 2255 3880 50  0000 R CNN
-F 2 "Diode_SMD:D_SOD-323_HandSoldering" V 2300 3950 50  0001 C CNN
+F 2 "Diode_SMD:D_SOD-128" V 2300 3950 50  0001 C CNN
 F 3 "~" V 2300 3950 50  0001 C CNN
 	1    2300 3950
@@
 F 0 "D23" V 2846 3880 50  0000 R CNN
 F 1 "D_Small" V 2755 3880 50  0000 R CNN
-F 2 "Diode_SMD:D_SOD-323_HandSoldering" V 2800 3950 50  0001 C CNN
+F 2 "Diode_SMD:D_SOD-128" V 2800 3950 50  0001 C CNN
 F 3 "~" V 2800 3950 50  0001 C CNN
 	1    2800 3950
@@
 F 0 "D24" V 3346 3880 50  0000 R CNN
 F 1 "D_Small" V 3255 3880 50  0000 R CNN
-F 2 "Diode_SMD:D_SOD-323_HandSoldering" V 3300 3950 50  0001 C CNN
+F 2 "Diode_SMD:D_SOD-128" V 3300 3950 50  0001 C CNN
 F 3 "~" V 3300 3950 50  0001 C CNN
 	1    3300 3950
@@
 F 0 "D25" V 3846 3880 50  0000 R CNN
 F 1 "D_Small" V 3755 3880 50  0000 R CNN
-F 2 "Diode_SMD:D_SOD-323_HandSoldering" V 3800 3950 50  0001 C CNN
+F 2 "Diode_SMD:D_SOD-128" V 3800 3950 50  0001 C CNN
 F 3 "~" V 3800 3950 50  0001 C CNN
 	1    3800 3950
@@
 F 0 "D26" V 4346 3880 50  0000 R CNN
 F 1 "D_Small" V 4255 3880 50  0000 R CNN
-F 2 "Diode_SMD:D_SOD-323_HandSoldering" V 4300 3950 50  0001 C CNN
+F 2 "Diode_SMD:D_SOD-128" V 4300 3950 50  0001 C CNN
 F 3 "~" V 4300 3950 50  0001 C CNN
 	1    4300 3950
@@
 F 0 "D27" V 4846 3880 50  0000 R CNN
 F 1 "D_Small" V 4755 3880 50  0000 R CNN
-F 2 "Diode_SMD:D_SOD-323_HandSoldering" V 4800 3950 50  0001 C CNN
+F 2 "Diode_SMD:D_SOD-128" V 4800 3950 50  0001 C CNN
 F 3 "~" V 4800 3950 50  0001 C CNN
 	1    4800 3950
@@
 F 0 "D28" V 5346 3880 50  0000 R CNN
 F 1 "D_Small" V 5255 3880 50  0000 R CNN
-F 2 "Diode_SMD:D_SOD-323_HandSoldering" V 5300 3950 50  0001 C CNN
+F 2 "Diode_SMD:D_SOD-128" V 5300 3950 50  0001 C CNN
 F 3 "~" V 5300 3950 50  0001 C CNN
 	1    5300 3950
@@
 F 0 "D29" V 5846 3880 50  0000 R CNN
 F 1 "D_Small" V 5755 3880 50  0000 R CNN
-F 2 "Diode_SMD:D_SOD-323_HandSoldering" V 5800 3950 50  0001 C CNN
+F 2 "Diode_SMD:D_SOD-128" V 5800 3950 50  0001 C CNN
 F 3 "~" V 5800 3950 50  0001 C CNN
 	1    5800 3950
@@
 F 0 "D30" V 6346 3880 50  0000 R CNN
 F 1 "D_Small" V 6255 3880 50  0000 R CNN
-F 2 "Diode_SMD:D_SOD-323_HandSoldering" V 6300 3950 50  0001 C CNN
+F 2 "Diode_SMD:D_SOD-128" V 6300 3950 50  0001 C CNN
 F 3 "~" V 6300 3950 50  0001 C CNN
 	1    6300 3950
@@
 F 0 "D31" V 3346 4530 50  0000 R CNN
 F 1 "D_Small" V 3255 4530 50  0000 R CNN
-F 2 "Diode_SMD:D_SOD-323_HandSoldering" V 3300 4600 50  0001 C CNN
+F 2 "Diode_SMD:D_SOD-128" V 3300 4600 50  0001 C CNN
 F 3 "~" V 3300 4600 50  0001 C CNN
 	1    3300 4600
@@
 F 0 "D32" V 3846 4530 50  0000 R CNN
 F 1 "D_Small" V 3755 4530 50  0000 R CNN
-F 2 "Diode_SMD:D_SOD-323_HandSoldering" V 3800 4600 50  0001 C CNN
+F 2 "Diode_SMD:D_SOD-128" V 3800 4600 50  0001 C CNN
 F 3 "~" V 3800 4600 50  0001 C CNN
 	1    3800 4600
@@
 F 0 "D33" V 4346 4530 50  0000 R CNN
 F 1 "D_Small" V 4255 4530 50  0000 R CNN
-F 2 "Diode_SMD:D_SOD-323_HandSoldering" V 4300 4600 50  0001 C CNN
+F 2 "Diode_SMD:D_SOD-128" V 4300 4600 50  0001 C CNN
 F 3 "~" V 4300 4600 50  0001 C CNN
 	1    4300 4600
@@
 F 0 "D34" V 4846 4530 50  0000 R CNN
 F 1 "D_Small" V 4755 4530 50  0000 R CNN
-F 2 "Diode_SMD:D_SOD-323_HandSoldering" V 4800 4600 50  0001 C CNN
+F 2 "Diode_SMD:D_SOD-128" V 4800 4600 50  0001 C CNN
 F 3 "~" V 4800 4600 50  0001 C CNN
 	1    4800 4600
